File: Programmer/Programmer.sch (KiCad schematic (older format))
At the start: 17 parts, among them J1 USB_C_Receptacle_USB2.0, J2 Prog, Q1 BC846BS, U1 AP2112K-3.3, U2 FT232RL-REEL

Commit message: Rettelse på programmer vcc
Connections:
- net +3V3: no longer U2.4 (VCCIO)
- net GNDD: now also J1.S1 (SHIELD)
- net VCC: now reaches C4.1, U2.17 (3V3OUT)
- net VCC: now also U2.19 (RESET), U2.4 (VCCIO)
- no-connect marks 1 -> 0
Other:
- moved on the sheet: D1, R3, R4
Changed lines of the file:
@@
 Connection ~ 5200 1050
-$Comp
-L power:+3V3 #PWR0107
-U 1 1 5F29D17D
-P 4950 2000
-F 0 "#PWR0107" H 4950 1850 50  0001 C CNN
-F 1 "+3V3" H 4965 2173 50  0000 C CNN
-F 2 "" H 4950 2000 50  0001 C CNN
-F 3 "" H 4950 2000 50  0001 C CNN
-	1    4950 2000
-	1    0    0    -1
-$EndComp
 $Comp
 L power:+5V #PWR0108
@@
 	3850 1050 3850 1250
 Wire Wire Line
-	4100 2000 4200 2000
-Wire Wire Line
-	4200 2000 4200 1600
-Wire Wire Line
-	4200 1600 3500 1600
-Wire Wire Line
-	3500 1600 3500 1050
-Wire Wire Line
 	3500 1050 3850 1050
 Connection ~ 3850 1050
@@
 	1    0    0    -1
 $EndComp
-NoConn ~ 1200 6200
 $Comp
 L power:GNDD #PWR0110
@@
 L Device:R_Small R3
 U 1 1 5F2A90CC
-P 3050 6050
-F 0 "R3" V 2854 6050 50  0000 C CNN
-F 1 "5k1" V 2945 6050 50  0000 C CNN
-F 2 "Resistor_SMD:R_0805_2012Metric" H 3050 6050 50  0001 C CNN
-F 3 "~" H 3050 6050 50  0001 C CNN
-	1    3050 6050
+P 3050 5800
+F 0 "R3" V 2854 5800 50  0000 C CNN
+F 1 "5k1" V 2945 5800 50  0000 C CNN
+F 2 "Resistor_SMD:R_0805_2012Metric" H 3050 5800 50  0001 C CNN
+F 3 "~" H 3050 5800 50  0001 C CNN
+	1    3050 5800
 	0    -1   -1   0
 $EndComp
@@
 L Device:R_Small R4
 U 1 1 5F2A9F6E
-P 3050 5050
-F 0 "R4" V 2854 5050 50  0000 C CNN
-F 1 "5k1" V 2945 5050 50  0000 C CNN
-F 2 "Resistor_SMD:R_0805_2012Metric" H 3050 5050 50  0001 C CNN
-F 3 "~" H 3050 5050 50  0001 C CNN
-	1    3050 5050
+P 3050 4800
+F 0 "R4" V 2854 4800 50  0000 C CNN
+F 1 "5k1" V 2945 4800 50  0000 C CNN
+F 2 "Resistor_SMD:R_0805_2012Metric" H 3050 4800 50  0001 C CNN
+F 3 "~" H 3050 4800 50  0001 C CNN
+	1    3050 4800
 	0    -1   -1   0
 $EndComp
@@
 	2450 5000 2400 5000
 Connection ~ 2400 5000
-Text GLabel 3550 6050 3    50   Input ~ 0
+Text GLabel 3550 5800 3    50   Input ~ 0
 D+
-Text GLabel 3550 5050 1    50   Input ~ 0
+Text GLabel 3550 4800 1    50   Input ~ 0
 D-
 Text GLabel 4100 2300 0    50   Input ~ 0
@@
 L dk_TVS-Diodes:USBLC6-2SC6 D1
 U 1 1 5F282DC2
-P 3850 5550
-F 0 "D1" V 3903 5022 60  0000 R CNN
-F 1 "824014" V 3797 5022 60  0000 R CNN
-F 2 "Package_TO_SOT_SMD:SOT-23-6" H 4050 5750 60  0001 L CNN
-F 3 "http://www.st.com/content/ccc/resource/technical/document/datasheet/06/1d/48/9c/6c/20/4a/b2/CD00050750.pdf/files/CD00050750.pdf/jcr:content/translations/en.CD00050750.pdf" H 4050 5850 60  0001 L CNN
-F 4 "497-5235-1-ND" H 4050 5950 60  0001 L CNN "Digi-Key_PN"
-F 5 "USBLC6-2SC6" H 4050 6050 60  0001 L CNN "MPN"
-F 6 "Circuit Protection" H 4050 6150 60  0001 L CNN "Category"
-F 7 "TVS - Diodes" H 4050 6250 60  0001 L CNN "Family"
-F 8 "http://www.st.com/content/ccc/resource/technical/document/datasheet/06/1d/48/9c/6c/20/4a/b2/CD00050750.pdf/files/CD00050750.pdf/jcr:content/translations/en.CD00050750.pdf" H 4050 6350 60  0001 L CNN "DK_Datasheet_Link"
-F 9 "/product-detail/en/stmicroelectronics/USBLC6-2SC6/497-5235-1-ND/1121688" H 4050 6450 60  0001 L CNN "DK_Detail_Page"
-F 10 "TVS DIODE 5.25V 17V SOT23-6" H 4050 6550 60  0001 L CNN "Description"
-F 11 "STMicroelectronics" H 4050 6650 60  0001 L CNN "Manufacturer"
-F 12 "Active" H 4050 6750 60  0001 L CNN "Status"
-	1    3850 5550
+P 3850 5300
+F 0 "D1" V 3903 4772 60  0000 R CNN
+F 1 "824014" V 3797 4772 60  0000 R CNN
+F 2 "Package_TO_SOT_SMD:SOT-23-6" H 4050 5500 60  0001 L CNN
+F 3 "http://www.st.com/content/ccc/resource/technical/document/datasheet/06/1d/48/9c/6c/20/4a/b2/CD00050750.pdf/files/CD00050750.pdf/jcr:content/translations/en.CD00050750.pdf" H 4050 5600 60  0001 L CNN
+F 4 "497-5235-1-ND" H 4050 5700 60  0001 L CNN "Digi-Key_PN"
+F 5 "USBLC6-2SC6" H 4050 5800 60  0001 L CNN "MPN"
+F 6 "Circuit Protection" H 4050 5900 60  0001 L CNN "Category"
+F 7 "TVS - Diodes" H 4050 6000 60  0001 L CNN "Family"
+F 8 "http://www.st.com/content/ccc/resource/technical/document/datasheet/06/1d/48/9c/6c/20/4a/b2/CD00050750.pdf/files/CD00050750.pdf/jcr:content/translations/en.CD00050750.pdf" H 4050 6100 60  0001 L CNN "DK_Datasheet_Link"
+F 9 "/product-detail/en/stmicroelectronics/USBLC6-2SC6/497-5235-1-ND/1121688" H 4050 6200 60  0001 L CNN "DK_Detail_Page"
+F 10 "TVS DIODE 5.25V 17V SOT23-6" H 4050 6300 60  0001 L CNN "Description"
+F 11 "STMicroelectronics" H 4050 6400 60  0001 L CNN "Manufacturer"
+F 12 "Active" H 4050 6500 60  0001 L CNN "Status"
+	1    3850 5300
 	0    -1   -1   0
 $EndComp
 Wire Wire Line
-	3550 6050 3150 6050
-Wire Wire Line
-	3550 5050 3150 5050
-Wire Wire Line
-	2950 6050 2950 5400
+	3550 5800 3150 5800
+Wire Wire Line
+	3550 4800 3150 4800
 Wire Wire Line
 	2100 5400 2950 5400
 Wire Wire Line
 	2100 5200 2950 5200
-Wire Wire Line
-	2950 5200 2950 5050
 $Comp
 L power:GNDD #PWR0112
 U 1 1 5F29BCC2
-P 3850 6050
-F 0 "#PWR0112" H 3850 5800 50  0001 C CNN
-F 1 "GNDD" H 3854 5895 50  0000 C CNN
-F 2 "" H 3850 6050 50  0001 C CNN
-F 3 "" H 3850 6050 50  0001 C CNN
-	1    3850 6050
-	1    0    0    -1
-$EndComp
-Text GLabel 3850 4750 2    50   Input ~ 0
+P 3850 5800
+F 0 "#PWR0112" H 3850 5550 50  0001 C CNN
+F 1 "GNDD" H 3854 5645 50  0000 C CNN
+F 2 "" H 3850 5800 50  0001 C CNN
+F 3 "" H 3850 5800 50  0001 C CNN
+	1    3850 5800
+	1    0    0    -1
+$EndComp
+Text GLabel 3850 4500 2    50   Input ~ 0
 VBUS
 Wire Wire Line
-	3850 5050 3850 4750
+	3850 4800 3850 4500
 Text Label 2650 5200 0    50   ~ 0
 D_N
 Text Label 2650 5400 0    50   ~ 0
 D_P
+Wire Wire Line
+	2950 4800 2950 5200
+Wire Wire Line
+	2950 5400 2950 5800
+$Comp
+L power:VCC #PWR?
+U 1 1 5F293AE4
+P 6150 2400
+F 0 "#PWR?" H 6150 2250 50  0001 C CNN
+F 1 "VCC" H 6165 2573 50  0000 C CNN
+F 2 "" H 6150 2400 50  0001 C CNN
+F 3 "" H 6150 2400 50  0001 C CNN
+	1    6150 2400
+	1    0    0    -1
+$EndComp
+Connection ~ 6150 2400
+$Comp
+L power:VCC #PWR?
+U 1 1 5F2941D3
+P 4950 2000
+F 0 "#PWR?" H 4950 1850 50  0001 C CNN
+F 1 "VCC" H 4965 2173 50  0000 C CNN
+F 2 "" H 4950 2000 50  0001 C CNN
+F 3 "" H 4950 2000 50  0001 C CNN
+	1    4950 2000
+	1    0    0    -1
+$EndComp
+$Comp
+L power:VCC #PWR?
+U 1 1 5F29487B
+P 4300 2050
+F 0 "#PWR?" H 4300 1900 50  0001 C CNN
+F 1 "VCC" H 4315 2223 50  0000 C CNN
+F 2 "" H 4300 2050 50  0001 C CNN
+F 3 "" H 4300 2050 50  0001 C CNN
+	1    4300 2050
+	1    0    0    -1
+$EndComp
+Wire Wire Line
+	4450 2400 4300 2400
+Wire Wire Line
+	4300 2400 4300 2050
+$Comp
+L power:GNDD #PWR?
+U 1 1 5F296ACA
+P 1200 6200
+F 0 "#PWR?" H 1200 5950 50  0001 C CNN
+F 1 "GNDD" H 1204 6045 50  0000 C CNN
+F 2 "" H 1200 6200 50  0001 C CNN
+F 3 "" H 1200 6200 50  0001 C CNN
+	1    1200 6200
+	1    0    0    -1
+$EndComp
 $EndSCHEMATC

Commit message: knap tilføjet
Parts:
- added D2, D3: LED, LED_SMD:LED_0805_2012Metric, symbol Device:LED
- added R7, R8: 1k, Resistor_SMD:R_0805_2012Metric, symbol Device:R_Small
Connections:
- net VCC: now also R7.2, R8.2
- net at U2.22 (CBUS1): now also D2.1 (K)
- net at U2.23 (CBUS0): now also D3.1 (K)
- new net: D2.2 (A), R7.1
- new net: D3.2 (A), R8.1
Changed lines of the file:
@@
 	2950 5400 2950 5800
 $Comp
-L power:VCC #PWR?
+L power:VCC #PWR0107
 U 1 1 5F293AE4
 P 6150 2400
-F 0 "#PWR?" H 6150 2250 50  0001 C CNN
+F 0 "#PWR0107" H 6150 2250 50  0001 C CNN
 F 1 "VCC" H 6165 2573 50  0000 C CNN
 F 2 "" H 6150 2400 50  0001 C CNN
@@
 Connection ~ 6150 2400
 $Comp
-L power:VCC #PWR?
+L power:VCC #PWR0113
 U 1 1 5F2941D3
 P 4950 2000
-F 0 "#PWR?" H 4950 1850 50  0001 C CNN
+F 0 "#PWR0113" H 4950 1850 50  0001 C CNN
 F 1 "VCC" H 4965 2173 50  0000 C CNN
 F 2 "" H 4950 2000 50  0001 C CNN
@@
 $EndComp
 $Comp
-L power:VCC #PWR?
+L power:VCC #PWR0114
 U 1 1 5F29487B
 P 4300 2050
-F 0 "#PWR?" H 4300 1900 50  0001 C CNN
+F 0 "#PWR0114" H 4300 1900 50  0001 C CNN
 F 1 "VCC" H 4315 2223 50  0000 C CNN
 F 2 "" H 4300 2050 50  0001 C CNN
@@
 	4300 2400 4300 2050
 $Comp
-L power:GNDD #PWR?
+L power:GNDD #PWR0115
 U 1 1 5F296ACA
 P 1200 6200
-F 0 "#PWR?" H 1200 5950 50  0001 C CNN
+F 0 "#PWR0115" H 1200 5950 50  0001 C CNN
 F 1 "GNDD" H 1204 6045 50  0000 C CNN
 F 2 "" H 1200 6200 50  0001 C CNN
@@
 	1    0    0    -1
 $EndComp
+$Comp
+L Device:LED D2
+U 1 1 5F292408
+P 3900 3250
+F 0 "D2" H 3893 2995 50  0000 C CNN
+F 1 "LED" H 3893 3086 50  0000 C CNN
+F 2 "LED_SMD:LED_0805_2012Metric" H 3900 3250 50  0001 C CNN
+F 3 "~" H 3900 3250 50  0001 C CNN
+	1    3900 3250
+	-1   0    0    1
+$EndComp
+$Comp
+L Device:LED D3
+U 1 1 5F29367C
+P 3900 3500
+F 0 "D3" H 3893 3245 50  0000 C CNN
+F 1 "LED" H 3893 3336 50  0000 C CNN
+F 2 "LED_SMD:LED_0805_2012Metric" H 3900 3500 50  0001 C CNN
+F 3 "~" H 3900 3500 50  0001 C CNN
+	1    3900 3500
+	-1   0    0    1
+$EndComp
+$Comp
+L Device:R_Small R7
+U 1 1 5F293E23
+P 3500 3250
+F 0 "R7" V 3304 3250 50  0000 C CNN
+F 1 "1k" V 3395 3250 50  0000 C CNN
+F 2 "Resistor_SMD:R_0805_2012Metric" H 3500 3250 50  0001 C CNN
+F 3 "~" H 3500 3250 50  0001 C CNN
+	1    3500 3250
+	0    1    1    0
+$EndComp
+Wire Wire Line
+	4450 3400 4050 3400
+Wire Wire Line
+	4050 3400 4050 3250
+Wire Wire Line
+	4450 3500 4050 3500
+$Comp
+L Device:R_Small R8
+U 1 1 5F29741C
+P 3500 3500
+F 0 "R8" V 3304 3500 50  0000 C CNN
+F 1 "1k" V 3395 3500 50  0000 C CNN
+F 2 "Resistor_SMD:R_0805_2012Metric" H 3500 3500 50  0001 C CNN
+F 3 "~" H 3500 3500 50  0001 C CNN
+	1    3500 3500
+	0    1    1    0
+$EndComp
+Wire Wire Line
+	3750 3500 3600 3500
+Wire Wire Line
+	3750 3250 3600 3250
+Wire Wire Line
+	3400 3500 3200 3500
+Wire Wire Line
+	3200 3500 3200 3250
+Wire Wire Line
+	3400 3250 3200 3250
+$Comp
+L power:VCC #PWR?
+U 1 1 5F2A9A67
+P 3200 3250
+F 0 "#PWR?" H 3200 3100 50  0001 C CNN
+F 1 "VCC" H 3215 3423 50  0000 C CNN
+F 2 "" H 3200 3250 50  0001 C CNN
+F 3 "" H 3200 3250 50  0001 C CNN
+	1    3200 3250
+	1    0    0    -1
+$EndComp
+Connection ~ 3200 3250
 $EndSCHEMATC
